File: pcb/ver0.1/OV2640_spi-flash_SRAM.sch (KiCad schematic (older format))
At the start: 18 parts, among them J5 629105136821, Q1 DMP3125L, U1 AP7312-1233W6-7, U2 AP7312-1828W6-7

Commit message: schematic changes updated
Parts:
- removed C1, C3: 10uF, Capacitor_SMD:C_0603_1608Metric, symbol fpga-play-rescue:C_Small-Device
- removed C2, C4, C5, C6: 1uF, Capacitor_SMD:C_0603_1608Metric, symbol fpga-play-rescue:C_Small-Device
- removed D4: USBLC6-2SC6, fpga-play:SOT95P280X145-6N, symbol fpga-play-rescue:USBLC6-2SC6-fpga-play
- removed D5: MBR120, Diode_SMD:D_SOD-123, symbol fpga-play-rescue:D_Schottky_Small-Device
- removed G1: logo, fpga-play:EL_logo, symbol fpga-play:logo
- removed J5: 629105136821, fpga-play:WE_629105136821, symbol fpga-play-rescue:629105136821-fpga-play
- removed Q1: DMP3125L, Package_TO_SOT_SMD:SOT-23, symbol fpga-play-rescue:Q_PMOS_GSD-Device
- removed R10: 1M, Resistor_SMD:R_0603_1608Metric, symbol fpga-play-rescue:R_Small-Device
- removed R12: 1.5K, Resistor_SMD:R_0603_1608Metric, symbol fpga-play-rescue:R_Small-Device
- removed R7: 10K, Resistor_SMD:R_0603_1608Metric, symbol fpga-play-rescue:R_Small-Device
- removed R8, R9: 22R, Resistor_SMD:R_0603_1608Metric, symbol fpga-play-rescue:R_Small-Device
- removed U1: AP7312-1233W6-7, Package_TO_SOT_SMD:SOT-23-6, symbol fpga-play:AP7312-1233W6-7
- removed U2: AP7312-1828W6-7, Package_TO_SOT_SMD:SOT-23-6, symbol fpga-play:AP7312-1828W6-7
- added C25, C26, C29, C7, C8: 0.1uF, Capacitor_SMD:C_0603_1608Metric, symbol fpga-play-rescue:C_Small-Device
- added J4: OV_2640, fpga-play:68712414522, symbol fpga-play-rescue:OV_2640-fpga-play
- added JP1, JP2, JP3, JP5: SolderJumper_2_Bridged, fpga-play:shorting_jumper-0402, symbol fpga-play-rescue:SolderJumper_2_Bridged-Jumper
- added R11, R13, R14, R15, R16, R18, R6: 10K, Resistor_SMD:R_0603_1608Metric, symbol fpga-play-rescue:R_Small-Device
- added U6: W25Q32JVSSIQ, Package_SO:SOIC-8_5.23x5.23mm_P1.27mm, symbol fpga-play-rescue:W25Q32JVSSIQ-fpga-play
- added U7: APS6404L, Package_SO:SOIC-8_3.9x4.9mm_P1.27mm, symbol fpga-play-rescue:ESP-PSRAM64-fpga-play
Connections:
- net +2V8: now also C7.1, C8.1, J4.10 (DVDD), J4.4 (AVDD)
- net +3V3: now also C25.1, C26.1, R11.2, R13.2, R14.2, R18.2, R6.2, U6.8 (VCC), U7.8 (VCC)
- net GND: now also C25.2, C26.2, C29.2, C7.2, C8.2, J4.15 (DGND), J4.2 (DGND), U6.4 (GND), U7.4 (VSS)
- net VDD: now also C29.1, J4.11 (DOVDD), R15.2, R16.2
- new net: JP5.1 (A), R6.1, U7.1 (~CE)
- new net: JP1.1 (A), R13.1, U6.1 (~CS~)
- new net Flash_MISO(PSRAM_SIO1): JP3.2 (B), U6.2 (DO(IO1)), U7.2 (SO/SIO(1))
- new net Flash_MOSI(PSRAM_SIO0): JP2.1 (A), U6.5 (DI(IO0)), U7.5 (SI/SIO(0))
- new net Flash_SCK(PSRAM_SCK): R11.1, U6.6 (CLK), U7.6 (SCLK)
- new net Flash_SS: JP1.2 (B)
- new net Flash_~HOLD~(PSRAM_SIO3): R18.1, U6.7 (~HOLD/!RST(IO3)~), U7.7 (SIO(3))
- new net Flash_~WP~(PSRAM_SIO2): R14.1, U6.3 (~WP(IO2)~), U7.3 (SIO(2))
- new net IOB_0A: J4.5 (SIO_C), R16.1
- new net IOB_2A: J4.23 (D1)
- new net IOB_3B_G6: J4.24 (D0)
- new net IOB_4A: J4.21 (D3)
- new net IOB_5B: J4.22 (D4)
- new net IOB_6A: J4.6 (RESET)
- new net IOB_9B: J4.20 (D5)
- new net IOT_13B: JP5.2 (B)
- new net IOT_36B: J4.8 (PWDN)
- new net IOT_37A: J4.7 (VSYNC)
- new net IOT_38B: J4.9 (HREF)
- new net IOT_39A: J4.12 (D9)
- new net IOT_41A: J4.13 (XCLK)
- new net IOT_42B: J4.14 (D8)
- new net IOT_43A: J4.16 (D7)
- new net IOT_44B: J4.17 (PCLK)
- new net IOT_45A_G1: J4.18 (D6)
- new net IOT_48B: J4.1 (STROBE)
- new net IOT_49A: J4.3 (STO_D), R15.1
- new net IOT_8A: J4.19 (D2)
- new net iCE_SI: JP3.1 (A)
- new net iCE_SO: JP2.2 (B)
Other:
- note added: "24 Pin FPC Connector"
- note added: "Flash Memory"
- note added: "For programming FPGA RAM"
- note added: "For programming FPGA RAM directly cut the 1-2 traces from \nJP2 and JP3 and connect them as 1-1 and 2-2."
- note added: "For programming Flash"
- note added: "JP1: Cut the 1-2 trace for programming FPGA RAM"
- note added: "PSRAM"
- note removed: "Input Voltage\n3.8V to 6.0V"
- note removed: "Power Supply"
- note removed: "USB Bootloader"
