File: pcb/ver0.1/OV7670_spi-flash_SRAM.sch (KiCad schematic (older format))
At the start: 18 parts, among them J4 687124183622, U6 W25Q32JVSSIQ, U7 ESP-PSRAM64

Commit message: schematic changes updated
Parts:
- removed C27, C28: 10uF, Capacitor_SMD:C_0603_1608Metric, symbol Device:C_Small
- removed J4: 687124183622, fpga-play:687124183622, symbol fpga-play:687124183622
- added C? (x2): 0.1uF, Capacitor_SMD:C_0603_1608Metric, symbol Device:C_Small
- added J?: OV_2640, symbol fpga-play-rescue:OV_2640-fpga-play
- C29: value 10uF -> 0.1uF
- U6: symbol fpga-play:W25Q32JVSSIQ -> fpga-play-rescue:W25Q32JVSSIQ-fpga-play
- U7: value ESP-PSRAM64 -> APS6404L; symbol fpga-play:ESP-PSRAM64 -> fpga-play-rescue:ESP-PSRAM64-fpga-play
Connections:
- net labels added: +1V8, +2V8, IOT_13B, IOT_36B, IOT_38B, IOT_39A, IOT_41A, IOT_42B, IOT_43A, IOT_44B, IOT_49A, VDD
- net labels removed: +3V0, IOB_20A, IOB_23B, IOB_24A, IOB_25B_G3, IOB_29B, IOB_31B, IOT_46B_G0, RGB2
- wire segments 109 -> 108
