File: pcb/ver0.1/fpga-play.kicad_pcb (KiCad board)
At the start: 2 copper layers, 32 x 63.8 mm, 69 parts, among them J1 IO Header, J2 Prog Header, J3 IO Header, J4 687124183622, J5 629105136821, Q1 DMP3125L, SW1 CRESET, SW2 User_Button, U1 TLV7111233DSET, U2 MIC5501-3.0YM5-TR, U4 SIT1602AC-12-33E-12.000000E, U5 ICE40UP5K-SG48ITR50, U6 W25Q32JVSSIQ, U7 ESP-PSRAM64

Commit message: schematic changes updated
Parts:
- removed C19, C20: 10nF, Capacitor_SMD:C_0603_1608Metric
- removed C27, C28: 10uF, Capacitor_SMD:C_0603_1608Metric
- removed U4: SIT1602AC-12-33E-12.000000E, fpga-play:SOIC254P1016X440-4N
- added C6: 1uF, Capacitor_SMD:C_0603_1608Metric, F.Cu at (137.6, 119.0)
- added C7: 0.1uF, Capacitor_SMD:C_0603_1608Metric, F.Cu at (133.2, 82.2)
- added C8: 0.1uF, Capacitor_SMD:C_0603_1608Metric, F.Cu at (136.6, 82.2)
- added D5: MBR120, Diode_SMD:D_SOD-123, F.Cu at (137.4, 122.4)
- added G1: logo, fpga-play:EL_logo, B.Cu at (138.7, 93.0)
- added JP4: Jumper_3_Bridged12, Connector_PinHeader_2.54mm:PinHeader_1x03_P2.54mm_Vertical, F.Cu at (147.8, 104.3)
- added JP5: SolderJumper_2_Bridged, fpga-play:shorting_jumper-0402, F.Cu at (150.2, 76.0)
- added R17: 10K, Resistor_SMD:R_0603_1608Metric, F.Cu at (144.6, 117.1)
- added R18: 10K, Resistor_SMD:R_0603_1608Metric, F.Cu at (142.5, 71.0)
- added Y1: DSC6101CI1A-012.0000T, fpga-play:DSC6101CI1A-012_0000T, F.Cu at (147.4, 116.2)
- C1, C3: value 1uF -> 10uF
- C18: value 10nF -> 0.1uF
- C29: value 10uF -> 0.1uF
- D1: value MBR130 -> 1N4148
- J1, J3: footprint Connector_PinHeader_2.54mm:PinHeader_1x18_P2.54mm_Vertical -> Connector_PinHeader_2.54mm:PinHeader_1x16_P2.54mm_Vertical
- J4: value 687124183622 -> OV_2640; footprint fpga-play:687124183622 -> fpga-play:68712414522
- JP1, JP2, JP3: footprint Resistor_SMD:R_0402_1005Metric -> fpga-play:shorting_jumper-0402
- R13, R14: value 22R -> 10K
- R8, R9: value 10K -> 22R
- U1: value TLV7111233DSET -> AP7312-1233W6-7; footprint fpga-play:SON50P150X150X80-6N -> Package_TO_SOT_SMD:SOT-23-6
- U2: value MIC5501-3.0YM5-TR -> AP7312-1828W6-7; footprint fpga-play:SOT95P280X145-5N -> Package_TO_SOT_SMD:SOT-23-6
- U7: value ESP-PSRAM64 -> APS6404L
- moved R14 56.4 mm to (138.2, 69.7)
- moved R8 52.3 mm to (145.4, 121.3), turned to 270 degrees
- moved R9 51.5 mm to (149.0, 121.3), turned to 270 degrees
- moved R13 51.1 mm to (138.2, 71.5)
- moved R7 49.8 mm to (139.7, 122.0), turned to 270 degrees
- moved R15 27.6 mm to (146.1, 109.5)
- moved R11 25.6 mm to (126.0, 71.0), turned to 270 degrees
- moved R16 25.0 mm to (146.1, 107.2)
- moved S1 18.0 mm to (136.9, 92.7), turned to 180 degrees
- moved C18 17.7 mm to (129.8, 110.2), turned to 180 degrees
- moved C1 11.0 mm to (128.0, 129.0), turned to 180 degrees
- moved R6 9.54 mm to (150.4, 74.4)
- moved C4 9.40 mm to (129.6, 119.8), turned to 180 degrees
- moved C9 8.45 mm to (144.6, 115.3)
- moved U2 6.74 mm to (133.6, 120.8), turned to 0 degrees
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Connections:
- C1 pad 1: +5V -> Net-(C1-Pad1)
- C12 pad 1: +3V3 -> VDD
- C13 pad 1: +3V3 -> VDD
- C15 pad 1: +3V3 -> +1V2
- C18 pad 1: +1V2 -> Net-(C18-Pad1)
- C22 pad 1: +3V3 -> VDD
- C24 pad 1: +3V3 -> VDD
- C29 pad 1: +3V0 -> VDD
- C3 pad 1: +5V -> Net-(C1-Pad1)
- C4 pad 1: +3V0 -> +2V8
- C9 pad 1: +3V3 -> VDD
- D1 pad 1: Net-(D1-Pad1) -> Net-(C18-Pad1)
- D4 pad 5: VDD -> VBUS
- J1 pad 10: IOB_29B -> IOT_43A
- J1 pad 11: IOB_25B_G3 -> IOB_31B
- J1 pad 12: IOB_23B -> IOB_29B
- J1 pad 13: IOT_37A -> IOB_25B_G3
- J1 pad 14: IOT_36B -> IOB_23B
- J1 pad 15: IOT_39A -> GND
- J1 pad 16: IOT_38B -> +3V3
- J1 pad 4: IOT_13B -> IOT_37A
- J1 pad 5: IOB_16A -> IOT_36B
- J1 pad 6: IOB_18A -> IOT_39A
- J1 pad 7: IOB_20A -> IOT_38B
- J1 pad 8: IOB_22A -> IOT_41A
- J1 pad 9: IOB_31B -> IOT_42B
- J2 pad 1: Flash_MOSI(PSRAM_SIO0) -> Flash_SS
- J2 pad 10: GND -> Flash_~WP~(PSRAM_SIO2)
- J2 pad 2: +3V3 -> GND
- J2 pad 3: Flash_SS -> Flash_SCK(PSRAM_SCK)
- J2 pad 4: Flash_~WP~(PSRAM_SIO2) -> +3V3
- J2 pad 5: ~CRESET_B -> Flash_MISO(PSRAM_SIO1)
- J2 pad 6: Flash_~HOLD~(PSRAM_SIO3) -> CDONE
- J2 pad 7: Flash_SCK(PSRAM_SCK) -> Flash_MOSI(PSRAM_SIO0)
- J2 pad 8: CDONE -> ~CRESET_B
- J2 pad 9: Flash_MISO(PSRAM_SIO1) -> Flash_~HOLD~(PSRAM_SIO3)
- J3 pad 10: IOT_45A_G1 -> IOT_50B
- J3 pad 11: IOT_48B -> IOT_45A_G1
- J3 pad 12: IOT_44B -> IOT_48B
- J3 pad 13: IOT_43A -> IOT_46B_G0
- J3 pad 14: IOT_42B -> IOT_44B
- J3 pad 15: IOT_41A -> GND
- J3 pad 16: +3V3 -> VCC
- J3 pad 8: Flash_~WP~(PSRAM_SIO2) -> RGB2
- J3 pad 9: IOT_50B -> RGB1
- J4 pad 1: Net-(J4-Pad1) -> IOT_48B
- J4 pad 10: +3V0 -> +2V8
- J4 pad 11: +3V0 -> VDD
- J4 pad 12: IOB_31B -> IOT_39A
- J4 pad 13: IOB_5B -> IOT_41A
- J4 pad 14: IOB_18A -> IOT_42B
- J4 pad 16: IOB_16A -> IOT_43A
- J4 pad 17: IOB_4A -> IOT_44B
- J4 pad 18: IOB_6A -> IOT_45A_G1
- J4 pad 19: IOB_29B -> IOT_8A
- J4 pad 20: IOB_2A -> IOB_9B
- J4 pad 21: IOT_8A -> IOB_4A
- J4 pad 22: IOB_25B_G3 -> IOB_5B
- J4 pad 23: IOT_37A -> IOB_2A
- J4 pad 24: IOT_48B -> IOB_3B_G6
- J4 pad 3: IOB_0A -> IOT_49A
- J4 pad 4: +3V0 -> +2V8
- J4 pad 5: IOB_3B_G6 -> IOB_0A
- J4 pad 6: IOB_9B -> IOB_6A
- J4 pad 7: IOB_24A -> IOT_37A
- J4 pad 8: IOB_23B -> IOT_36B
- J4 pad 9: IOB_20A -> IOT_38B
- J5 pad 1: VDD -> VBUS
- Q1 pad 1: GND -> VBUS
- Q1 pad 2: +5V -> Net-(C1-Pad1)
- Q1 pad 3: VDD -> VCC
- R11 pad 1: +3V3 -> Flash_SCK(PSRAM_SCK)
- R11 pad 2: IOT_45A_G1 -> +3V3
- R12 pad 1: IOT_45A_G1 -> +3V3
- R13 pad 1: Net-(D4-Pad6) -> Net-(JP1-Pad1)
- R13 pad 2: IOT_50B -> +3V3
- R14 pad 1: Net-(D4-Pad4) -> Flash_~WP~(PSRAM_SIO2)
- R14 pad 2: IOT_51A -> +3V3
- R15 pad 1: IOB_6A -> IOT_49A
- R15 pad 2: +3V3 -> VDD
- R16 pad 1: IOB_25B_G3 -> IOB_0A
- R16 pad 2: +3V3 -> VDD
- R6 pad 1: +3V3 -> Net-(JP5-Pad1)
- R6 pad 2: Flash_SCK(PSRAM_SCK) -> +3V3
- R7 pad 1: +3V3 -> VBUS
- R7 pad 2: Net-(JP1-Pad1) -> GND
- R8 pad 1: +3V3 -> USB_N
- R8 pad 2: Flash_~WP~(PSRAM_SIO2) -> Net-(D4-Pad6)
- R9 pad 1: +3V3 -> USB_P
- R9 pad 2: Flash_~HOLD~(PSRAM_SIO3) -> Net-(D4-Pad4)
- U1 pad 1: +5V -> +3V3
- U1 pad 2: +5V -> GND
- U1 pad 3: +5V -> Net-(C1-Pad1)
- U1 pad 4: GND -> Net-(C1-Pad1)
- U1 pad 5: +3V3 -> Net-(C1-Pad1)
- U2 pad 1: +5V -> +2V8
- U2 pad 3: +5V -> Net-(C1-Pad1)
- U2 pad 4: (no net) -> Net-(C1-Pad1)
- U2 pad 5: +3V0 -> Net-(C1-Pad1)
- U5 pad 1: +3V3 -> VDD
- U5 pad 10: IOB_18A -> Flash_~WP~(PSRAM_SIO2)
- U5 pad 11: IOB_20A -> /iCE40UP5K/SW1
- U5 pad 12: IOB_22A -> USB_P
- U5 pad 13: IOB_24A -> USB_N
- U5 pad 24: Net-(D1-Pad1) -> Net-(C18-Pad1)
- U5 pad 33: +3V3 -> VDD
- U5 pad 35: Flash_~HOLD~(PSRAM_SIO3) -> IOT_46B_G0
- U5 pad 40: /iCE40UP5K/SW1 -> RGB1
- U5 pad 41: Flash_~WP~(PSRAM_SIO2) -> RGB2
- U5 pad 9: IOB_16A -> Flash_~HOLD~(PSRAM_SIO3)
- U7 pad 1: IOT_45A_G1 -> Net-(JP5-Pad1)
Routing:
- net +3V3: track 244.6 -> 99.1 mm, vias 14 -> 18
- net +3V0: track 91.7 -> 0.00 mm, vias 4 -> 0
- net IOB_16A: track 54.9 -> 0.00 mm, vias 1 -> 0
- net IOT_43A: track 15.5 -> 65.3 mm, vias 0 -> 1
- net IOT_44B: track 14.7 -> 64.4 mm, vias 0 -> 1
- net IOB_25B_G3: track 67.3 -> 18.3 mm
- net Flash_~HOLD~(PSRAM_SIO3): track 118.2 -> 69.5 mm, vias 4 -> 3
- net IOB_18A: track 47.3 -> 0.00 mm, vias 1 -> 0
- net IOT_42B: track 17.7 -> 63.8 mm, vias 0 -> 1
- net IOB_20A: track 44.3 -> 0.00 mm, vias 1 -> 0
- net IOB_23B: track 61.0 -> 20.6 mm
- net IOB_29B: track 56.7 -> 16.3 mm
- net iCE_SO: track 73.9 -> 35.8 mm
- net IOB_24A: track 36.7 -> 0.00 mm, vias 2 -> 0
- net IOT_39A: track 18.0 -> 52.0 mm, vias 0 -> 1
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- added copper zone on F.Cu, net +1V8
- added copper zone on In2.Cu, net +1V8
- added copper zone on F.Cu, net +2V8
- added copper zone on In2.Cu, net +2V8
- added copper zone on B.Cu, net +3V3
- added copper zone on In2.Cu, net +3V3
- added copper zone on In1.Cu, net GND
- added copper zone on F.Cu, net Net-(C1-Pad1)
- added copper zone on In2.Cu, net Net-(C1-Pad1)
- added copper zone on B.Cu, net VBUS
- added copper zone on B.Cu, net VCC
- added copper zone on In2.Cu, net VDD
- removed copper zone on F.Cu, net +3V0
- removed copper zone on F.Cu, net +5V
- removed copper zone on B.Cu, net GND
- removed copper zone on F.Cu, net GND
Other:
- copper layers 2 -> 4
- board text added: "1V8"
- board text added: "35"
- board text added: "CRST"
- board text added: "HOLD"
- board text added: "MISO"
- board text added: "MOSI"
- board text added: "SS"
- board text added: "Ver 0.1"
- board text added: "WP"
- board text removed: "10"
- board text removed: "11"
- board text removed: "6"
- board text removed: "9"
- board text removed: "CS"
- board text removed: "SI"
- board text removed: "SO"
- board text removed: "~CRST"
- board text removed: "~HOLD"
- board text removed: "~WP"
