File: pcb/ver0.1/fpga-play.sch (KiCad schematic (older format))
At the start: 6 parts

Commit message: schematic changes updated
Parts:
- FID1, FID2, FID3: symbol Mechanical:Fiducial -> fpga-play-rescue:Fiducial-Mechanical
- H1, H2: symbol Mechanical:MountingHole -> fpga-play-rescue:MountingHole-Mechanical
- S1: symbol fpga-play:fpga_silk -> fpga-play-rescue:fpga_silk-fpga-play
