File: pcb/ver0.1/iCE40UP5K_SG48ITR.sch (KiCad schematic (older format))
At the start: 28 parts, among them SW1 CRESET, SW2 User_Button, U4 SIT1602AC-12-33E-12.000000E, U5 ICE40UP5K-SG48ITR50

Commit message: schematic changes updated
Parts:
- removed C15, C18, C19, C20: 10nF, Capacitor_SMD:C_0603_1608Metric, symbol Device:C_Small
- removed U4: SIT1602AC-12-33E-12.000000E, fpga-play:SOIC254P1016X440-4N, symbol fpga-play:SIT1602AC-12-33E-12.000000E
- added C15: 10nF, Capacitor_SMD:C_0603_1608Metric, symbol fpga-play-rescue:C_Small-Device
- added C18: 0.1uF, Capacitor_SMD:C_0603_1608Metric, symbol fpga-play-rescue:C_Small-Device
- added JP4: Jumper_3_Bridged12, Connector_PinHeader_2.54mm:PinHeader_1x03_P2.54mm_Vertical, symbol fpga-play-rescue:Jumper_3_Bridged12-Jumper
- added R17: 10K, Resistor_SMD:R_0603_1608Metric, symbol fpga-play-rescue:R_Small-Device
- added Y1: DSC6101CI1A-012.0000T, fpga-play:DSC6101CI1A-012_0000T, symbol fpga-play-rescue:DSC6101CI1A-012.0000T-fpga-play
- C10, C11, C12, C13, C14, C16, C17, C21, C22, C23, C24, C9: symbol Device:C_Small -> fpga-play-rescue:C_Small-Device
- D1: value MBR130 -> 1N4148; symbol Device:D_Small -> fpga-play-rescue:D_Small-Device
- D2, D3: symbol Device:LED_Small -> fpga-play-rescue:LED_Small-Device
- R1, R2, R3, R4, R5: symbol Device:R_Small -> fpga-play-rescue:R_Small-Device
- SW1, SW2: symbol Switch:SW_Push -> fpga-play-rescue:SW_Push-Switch
- U5: symbol fpga-play:ICE40UP5K-SG48ITR50 -> fpga-play-rescue:ICE40UP5K-SG48ITR50-fpga-play
Connections:
- net labels added: +1V8, RGB1, VDD
- net labels removed: IOB_20A, USB_DET, VCC
- wire segments 139 -> 132
Other:
- note added: "Bank 0&2 Voltage Selection"
- note added: "CDONE LED"
- note added: "CRESET Button"
- note added: "Crystal Osillator"
- note added: "Note:"
- note added: "User Button"
- note added: "User LED"
- note added: "While using the camera jumper must be on \npin 1 and 2."
