File: pcb/ver0.1/io_headers.sch (KiCad schematic (older format))
At the start: 3 parts, among them J1 IO Header, J2 Prog Header, J3 IO Header

Commit message: schematic changes updated
Parts:
- removed J1, J3: IO Header, Connector_PinHeader_2.54mm:PinHeader_1x18_P2.54mm_Vertical, symbol Connector_Generic:Conn_01x18
- added J1, J3: IO Header, Connector_PinHeader_2.54mm:PinHeader_1x16_P2.54mm_Vertical, symbol fpga-play-rescue:Conn_01x16-Connector_Generic
- J2: symbol Connector_Generic:Conn_02x05_Odd_Even -> fpga-play-rescue:Conn_02x05_Odd_Even-Connector_Generic
Connections:
- net labels added: IOT_46B_G0, RGB1, VCC
- net labels removed: IOB_16A, IOB_18A, IOB_20A, IOB_22A, IOT_13B, VDD
- wire segments 50 -> 45
